File: electronics/psu_battery_double_symmetrical/psu_battery_double_symmetrical.kicad_pcb (KiCad board)
At the start: 2 copper layers, 78.1 x 41.9 mm, 22 parts, among them J3 Conn_01x02, J4 Conn_01x02, SW1 switch_DPDT, U1 TSC432

Commit message: review done
Parts:
- moved LED1 0.12 mm to (170.3, 89.4)
Routing:
- net GND: vias 0 -> 2
Changed lines of the file:
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@@
   (net 35 "Net-(LED1-A2)")
   (footprint "SquantorDiodes:LED_DUAL_TH245_90deg" (layer "F.Cu")
-    (at 170.3 89.3 90)
+    (at 170.3 89.425 90)
     (property "Sheetfile" "psu_battery_double_symmetrical.kicad_sch")
     (property "Sheetname" "")
@@
     (property "ki_keywords" "Dual LED Common cathode")
     (attr through_hole)
-    (fp_text reference "LED1" (at 0 -2 90 unlocked) (layer "F.SilkS")
+    (fp_text reference "LED1" (at -5.4 -0.8 90 unlocked) (layer "F.SilkS")
         (effects (font (size 0.8 0.8) (thickness 0.15)))
     )
@@
     (property "Sheetname" "")
     (attr smd)
-    (fp_text reference "N3" (at 13.6 -32.4 90 unlocked) (layer "F.SilkS")
+    (fp_text reference "N3" (at 14.5 -28.7 90 unlocked) (layer "F.SilkS")
         (effects (font (size 0.8 0.8) (thickness 0.15)))
     )
@@
     (property "ki_keywords" "mounting hole")
     (attr exclude_from_pos_files)
-    (fp_text reference "H1" (at -3.81 -1.27) (layer "F.SilkS")
+    (fp_text reference "H1" (at -3.12 2.35) (layer "F.SilkS")
         (effects (font (size 1 1) (thickness 0.15)))
     )
@@
     (property "ki_keywords" "R res resistor")
     (attr smd)
-    (fp_text reference "R4" (at 0 1.2) (layer "B.SilkS")
-        (effects (font (size 0.8 0.8) (thickness 0.15)) (justify mirror))
-    )
-    (fp_text value "4K7" (at 0 -1.2) (layer "B.Fab")
+    (fp_text reference "R4" (at -0.85 1.1) (layer "B.SilkS")
+        (effects (font (size 0.8 0.8) (thickness 0.15)) (justify mirror))
+    )
+    (fp_text value "4K7" (at 1.35 1.1) (layer "B.SilkS")
         (effects (font (size 0.8 0.8) (thickness 0.15)) (justify mirror))
     )
@@
     (property "ki_keywords" "R res resistor")
     (attr smd)
-    (fp_text reference "R5" (at 0 1.2) (layer "B.SilkS")
-        (effects (font (size 0.8 0.8) (thickness 0.15)) (justify mirror))
-    )
-    (fp_text value "4K7" (at 0 -1.2) (layer "B.Fab")
+    (fp_text reference "R5" (at -0.8 1.1) (layer "B.SilkS")
+        (effects (font (size 0.8 0.8) (thickness 0.15)) (justify mirror))
+    )
+    (fp_text value "4K7" (at 1.4 1.1) (layer "B.SilkS")
         (effects (font (size 0.8 0.8) (thickness 0.15)) (justify mirror))
     )
@@
   (gr_line (start 175.895 121.285) (end 97.79 121.285)
     (stroke (width 0.05) (type default)) (layer "Edge.Cuts"))
+  (via (at 109.6 117.6) (size 0.7) (drill 0.3) (layers "F.Cu" "B.Cu") (free) (net 10))
+  (via (at 106.2 117.6) (size 0.7) (drill 0.3) (layers "F.Cu" "B.Cu") (free) (net 10))
   (segment (start 128.3 109.9) (end 133.7 109.9) (width 1) (layer "F.Cu") (net 23))
   (segment (start 134.1 109.9) (end 167 109.9) (width 1) (layer "F.Cu") (net 23))
@@
   (segment (start 168.85 86.7) (end 170.24 86.7) (width 0.4) (layer "B.Cu") (net 35))
   (zone (net 10) (net_name "GND") (layers "F&B.Cu") (hatch edge 0.5)
-    (connect_pads (clearance 0.508))
+    (connect_pads (clearance 0.3))
     (min_thickness 0.25) (filled_areas_thickness no)
-    (fill yes (thermal_gap 0.5) (thermal_bridge_width 0.5))
+    (fill yes (thermal_gap 0.2) (thermal_bridge_width 0.4))
     (polygon
       (pts

Commit message: prepared for production minor updates
Parts:
- N1: value 20240424 -> 20240426
Changed lines of the file:
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@@
         (effects (font (size 1 1) (thickness 0.15)) (justify mirror))
     )
-    (fp_text value "20240424" (at 0 0) (layer "B.SilkS")
+    (fp_text value "20240426" (at 0 0) (layer "B.SilkS")
         (effects (font (size 0.8 0.8) (thickness 0.15)) (justify mirror))
     )
