File: electronics/psu_battery_double_symmetrical/psu_battery_double_symmetrical.kicad_sch (KiCad schematic)
At the start: 22 parts, among them J3 Conn_01x02, J4 Conn_01x02, SW1 switch_DPDT, U1 TSC432

Commit message: prepared for production minor updates
Parts:
- N1: value 20240424 -> 20240426
Changed lines of the file:
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@@
       (effects (font (size 1.524 1.524)) (justify left))
     )
-    (property "Value" "20240424" (at 20.32 189.23 0)
+    (property "Value" "20240426" (at 20.32 189.23 0)
       (effects (font (size 1.524 1.524)) (justify left))
     )
